File: elec/layout/default/pca9615.kicad_pcb (KiCad board)
At the start: 2 copper layers, 225.7 x 100.8 mm, 0 parts

Commit message: initial publish
Parts:
- added R1: Chip Resistor - Surface Mount 300Ohms ±5% 1/10W 0603 RoHS, lib:R0603, F.Cu at (155.2, 91.0)
- added R2: Chip Resistor - Surface Mount 100Ohms ±5% 1/10W 0603 RoHS, lib:R0603, F.Cu at (155.2, 92.6)
- added R3: Chip Resistor - Surface Mount 300Ohms ±5% 1/10W 0603 RoHS, lib:R0603, F.Cu at (155.2, 94.2)
- added R4: Chip Resistor - Surface Mount 300Ohms ±5% 1/10W 0603 RoHS, lib:R0603, F.Cu at (155.2, 96.0)
- added R5: Chip Resistor - Surface Mount 100Ohms ±5% 1/10W 0603 RoHS, lib:R0603, F.Cu at (155.2, 97.8)
- added R6: Chip Resistor - Surface Mount 300Ohms ±5% 1/10W 0603 RoHS, lib:R0603, F.Cu at (155.2, 99.4)
- added U1: , lib:TSSOP-10_L3.0-W3.0-P0.50-LS4.9-BL, F.Cu at (149.4, 95.1)
Routing:
- net vdd_b_: track 0.00 -> 20.2 mm, vias 0 -> 4
- net dsdap: track 0.00 -> 14.0 mm, vias 0 -> 1
- net dsclm: track 0.00 -> 11.1 mm, vias 0 -> 1
- net dsdam: track 0.00 -> 10.4 mm, vias 0 -> 1
- net dsclp: track 0.00 -> 9.99 mm, vias 0 -> 1
- net scl: track 0.00 -> 2.55 mm, vias 0 -> 1
- net vdd_a_: track 0.00 -> 2.36 mm, vias 0 -> 1
- net en: track 0.00 -> 2.35 mm, vias 0 -> 1
- net sda: track 0.00 -> 2.15 mm, vias 0 -> 1
Other:
- board outline removed
- board text removed: "{{GITHASH}}"
